File: pcb/micromouse-pcb.kicad_sch (KiCad schematic)
At the start: 108 parts, among them J1 BATT_IN_2S, J10 TB6612_BREAKOUT_CTRL, J11 TB6612_BREAKOUT_PWR_OUT, J12 Arduino Nano ESP32 digital row, J13 Arduino Nano ESP32 analog row, J2 EXT_SWITCH, J3 BATT_BALANCE_2S, J4 NUCLEO-G431KB digital row (D1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, J5 MOTOR_A_N20_ENCODER, J6 MOTOR_B_N20_ENCODER, J8 NUCLEO-G431KB analog row (D13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, Q1 Q_PMOS (e.g. DMP2035U-7), Q10 SFH309, Q11 BSS138 (real part; Q_NMOS_GSD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, Q12 SFH309, Q13 BSS138 (real part; Q_NMOS_GSD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, Q14 SFH309, Q15 BSS138 (real part; Q_NMOS_GSD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, Q16 SFH309, Q17 BSS138 (real part; Q_NMOS_GSD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, Q18 SFH309, Q19 BSS138 (real part; Q_NMOS_GSD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, Q2 SFH309, Q20 SFH309, Q21 BSS138 (real part; Q_NMOS_GSD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, Q22 SFH309, Q23 BSS138 (real part; Q_NMOS_GSD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, Q24 SFH309, Q25 BSS138 (real part; Q_NMOS_GSD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, Q26 SFH309, Q27 BSS138 (real part; Q_NMOS_GSD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, Q28 SFH309, Q29 BSS138 (real part; Q_NMOS_GSD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, Q3 BSS138 (real part; Q_NMOS_GSD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, Q4 SFH309, Q5 BSS138 (real part; Q_NMOS_GSD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, Q6 SFH309, Q7 BSS138 (real part; Q_NMOS_GSD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, Q8 SFH309, Q9 BSS138 (real part; Q_NMOS_GSD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, SW1 SW_Push, U1 AP63203WU (fixed 3.3V; symbol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, U4 HEF4067BT, U5 HEF4067BT

Commit message: Rev 2: ESP32-only redesign -- 100x128mm, 4 layers, DRC-clean
Drop the STM32 entirely (user decision): one socketed Arduino Nano ESP32
(real Module:Arduino_Nano footprint, pad map locked to the USB marker)
now does all control + telemetry. All control nets kept their names and
moved to A1; ADC nets on A0-A2; UART flash relay removed.

Board shrinks 150x185 -> 100x128mm (chamfered, wheels inside via interior
slots). In-house router generalized to N layers (THT pierces all, SMD its
face, through-vias join, per-layer H/V discipline) + a 0.25mm fine-grid
retry pass: 2012 tracks / 150 vias on 4 signal layers, 5 edges left for
the GUI. ERC 0, DRC 0 errors.

Also: wall-sensor side clusters with rotated THT LEDs (fixes a real
THT-into-bottom-SMD short), castor hole moved out of the line array,
smaller buck inductor (SRP7028A), CONNECTIONS.md fully regenerated for
the ESP32-only design (96 nets, coverage-enforced).

Co-Authored-By: Claude Fable 5 <noreply@anthropic.com>
Parts:
- removed J12: Arduino Nano ESP32 digital row, Connector_PinSocket_2.54mm:PinSocket_1x15_P2.54mm_Vertical, symbol Connector_Generic:Conn_01x15
- removed J13: Arduino Nano ESP32 analog row, Connector_PinSocket_2.54mm:PinSocket_1x15_P2.54mm_Vertical, symbol Connector_Generic:Conn_01x15
- removed J4: NUCLEO-G431KB digital row (D12..D2,GND,RST,D0,D1), Connector_PinSocket_2.54mm:PinSocket_1x15_P2.54mm_Vertical, symbol Connector_Generic:Conn_01x15
- removed J8: NUCLEO-G431KB analog row (D13,3V3,AREF,A0..A7,5V,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, Connector_PinSocket_2.54mm:PinSocket_1x15_P2.54mm_Vertical, symbol Connector_Generic:Conn_01x15
- added A1: Arduino Nano ESP32 (ESP32-S3) -- sole controller,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, Module:Arduino_Nano, symbol Connector_Generic:Conn_02x15_Odd_Even
- L1: footprint Inductor_SMD:L_Bourns_SRR1260 -> Inductor_SMD:L_Bourns_SRP7028A_7.3x6.6mm
Connections:
- net AIN1: now also A1.22 (Pin_22)
- net AIN2: now also A1.23 (Pin_23)
- net BIN1: now also A1.24 (Pin_24)
- net BIN2: now also A1.25 (Pin_25)
- net ENC1_A: now also A1.16 (Pin_16)
- net ENC1_B: now also A1.17 (Pin_17)
- net ENC2_A: now also A1.18 (Pin_18)
- net ENC2_B: now also A1.19 (Pin_19)
- net GND: now also A1.10 (Pin_10), A1.11 (Pin_11), A1.14 (Pin_14), A1.2 (Pin_2), A1.27 (Pin_27), A1.5 (Pin_5)
- net LED_PULSE: now also A1.6 (Pin_6)
- net MUX_S0: now also A1.15 (Pin_15)
- net MUX_S1: now also A1.9 (Pin_9)
- net MUX_S2: now also A1.8 (Pin_8)
- net MUX_S3: now also A1.7 (Pin_7)
- net MUX_SENSE: now also A1.12 (Pin_12)
- net PWMA: now also A1.20 (Pin_20)
- net PWMB: now also A1.21 (Pin_21)
- net STBY: now also A1.26 (Pin_26)
- no-connect marks 31 -> 11
Other:
- note added: "+3V3 is the single regulated logic rail: the ESP32 dev board, mux logic, encoder VCC, phototransistor pull-ups, and IR LED driver current all come from here (not raw VM_BATT)."
- note added: "Breakout logic inputs: STBY, AIN1/AIN2, BIN1/BIN2 are plain ESP32 GPIO; PWMA/PWMB are ESP32 LEDC PWM outputs (firmware configures PWM). VM=raw battery, VCC=+3V3 logic, GND common. AO1/AO2 -> motor A (MOTA_P/N), BO1/BO2 -> motor B (MOTB_P/N). The breakout's own board carries VM/VCC decoupling. VERIFY the breakout's real pin order + row spacing before fab."
- note added: "CONTROLLER -- socketed Arduino Nano ESP32 (ESP32-S3): control + sensors + telemetry"
- note added: "Single ESP32-S3 runs everything: TB6612 (STBY/PWMA/PWMB/AIN*/BIN*), 4 encoder inputs, the 2x HEF4067 sensor muxes (MUX_S0-S3 select, MUX_SENSE ADC, LED_PULSE), the two battery-sense ADCs, and USER_BTN. Wi-Fi/BLE telemetry is built in; flashed over the board's own USB-C -- no separate programmer or UART relay. The 3 analog nets are on A0-A2 (real ADC pins). The Nano-ESP32 header-to-GPIO map, and w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"
- note added: "USER_BTN (ESP32 A7) -- active-low start-run button, pulled up to +3V3. Standard micromouse UX (arm, then start a run). One of the ESP32 analog-capable pins; the full net/pin allocation is in PROJECT_NOTES.md. No separate debug/programming header on this board: the Arduino Nano ESP32 is flashed over its own onboard USB-C, and firmware is updated the same way (or over-the-air via Wi-Fi). No BOOT0/S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"
- note added: "VBAT_CELL1_SENSE = cell1 voltage (0-4.2V) scaled to <=2.9V. VBAT_PACK_SENSE = full pack voltage (0-8.4V) scaled to <=3.3V. Firmware computes cell2 = pack - cell1. Both wired to ESP32 ADC pins A2/A1 (VBAT_PACK_SENSE/VBAT_CELL1_SENSE) -- see GPIO allocation table in PROJECT_NOTES.md."
- note removed: "+3V3 is the single regulated logic rail: STM32, ESP32, mux logic, encoder VCC, phototransistor pull-ups, and IR LED driver current all come from here (not raw VM_BATT)."
- note removed: "BOOT0 and SWD (PA13/PA14) are NOT on the Nano header rows on this board -- confirmed against ST documentation (UM2397 family). Wireless STM32 update uses a firmware-level System-Memory-bootloader jump (AN2606) triggered over UART, not a hardware BOOT0 line -- see PROJECT_NOTES.md. NRST is on the header (both rows carry a reset pin, same physical line), also driven by an ESP32 GPIO (open-drain) fo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"
- note removed: "Breakout logic inputs: STBY, AIN1/AIN2, BIN1/BIN2 are plain STM32 GPIO; PWMA/PWMB are TIM1_CH1/CH4 (firmware configures PWM). VM=raw battery, VCC=+3V3 logic, GND common. AO1/AO2 -> motor A (MOTA_P/N), BO1/BO2 -> motor B (MOTB_P/N). The breakout's own board carries VM/VCC decoupling. VERIFY the breakout's real pin order + row spacing before fab."
- note removed: "MCU -- NUCLEO-G431KB socketed via two Nano-compatible 1x15 headers (CN3 + CN4)"
- note removed: "Only 5 pins used: 3V3 (power in from our rail -- do NOT also power via the board's USB while battery is on), GND, D0/RX <- STM32 USART1_TX, D1/TX -> STM32 USART1_RX, and D2 -> STM32 NRST (firmware open-drain, so it never fights the Nucleo's own reset). Everything else on the dev board (USB, auto-reset, boot button, regulator) is onboard, so the SMD version's strap buttons / programming header / d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"
- note removed: "USER_BTN (PA2/A7) -- active-low start-run button, pulled up to +3V3. This is the one Nano-header pin left over once every other net was assigned -- the GPIO budget across the 22 usable signal pins came out exactly even otherwise (see the full allocation table in PROJECT_NOTES.md). Not in the original spec, added because the pin was there and a start button is standard micromouse UX. No SWD/BOOT0 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"
- note removed: "VBAT_CELL1_SENSE = cell1 voltage (0-4.2V) scaled to <=2.9V. VBAT_PACK_SENSE = full pack voltage (0-8.4V) scaled to <=3.3V. Firmware computes cell2 = pack - cell1. Both wired to MCU ADC pins D8/D7 (PF1/PF0) -- see final GPIO allocation table in PROJECT_NOTES.md."
- note removed: "WIRELESS -- socketed Arduino Nano ESP32 dev board (telemetry + STM32 update relay)"

Commit message: Rev 3: line indicator LEDs, research-verified sensor geometry, 100x114mm
User requests: per-channel indicator LEDs on top, professional wall-sensor
positioning, smaller/tighter board.

- 8 indicator LEDs (D15-D22 + 1k + BSS138, gate on each LINEx_SENSE):
  zero DC load on the analog nodes; crisp threshold indication (LED ON =
  dark line). Adversarial review caught duty-cycle blindness (pulsed
  emitters leave nodes ambient-dominated ~93% of the time) -- fixed by
  dropping line emitters 33R -> 120R (~15mA) so firmware can latch all 8
  on continuously in line-follow mode. BOM: super-red AlInGaP indicators
  + daylight-filtered line receivers REQUIRED (optical feedback).

- Wall sensors repositioned per primary-source research (Harrison Decimus,
  UKMARS, Zeetah): front pair (toe-out) 89mm ahead of the axle, 45-deg
  diagonals ON the chamfered corners 74mm, side pair (forward toe) 56mm --
  all well in front of the center of rotation, per the verbatim Decimus
  6-sensor doctrine. Assembly aiming/shielding notes in PROJECT_NOTES.

- Board 100x128 -> 100x114: controller rotated horizontal, muxes to the
  side edges, axle forward to y=92, mounting holes added as router
  obstacles. 2139 tracks / 179 vias on 4 layers, ERC 0, DRC 0 errors,
  9 edges left for GUI finishing.

Co-Authored-By: Claude Fable 5 <noreply@anthropic.com>
Parts:
- added D15, D16, D17, D18, D19, D20, D21, D22: Indicator LED 0603 super-red AlInGaP, high-effici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, LED_SMD:LED_0603_1608Metric, symbol LED:LD271
- added Q30, Q31, Q32, Q33, Q34, Q35, Q36, Q37: BSS138 (real part; Q_NMOS_GSD base symbol used so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, Package_TO_SOT_SMD:SOT-23, symbol Transistor_FET:Q_NMOS_GSD
- added R41, R42, R43, R44, R45, R46, R47, R48: 1k, Resistor_SMD:R_0805_2012Metric, symbol Device:R
- R26, R28, R30, R32, R34, R36, R38, R40: value 33 -> 120
Connections:
- net GND: now also D18.1 (K), D18.2 (A), D20.2 (A), D21.1 (K), Q30.2 (S), Q31.2 (S), Q32.1 (G), Q32.2 (S), Q33.1 (G), Q33.2 (S), Q33.3 (D), Q34.1 (G), Q34.2 (S), Q35.2 (S), Q36.1 (G), Q36.2 (S), Q36.3 (D), Q37.1 (G), Q37.2 (S), R41.1, R42.1, R43.1, R44.1, R44.2, R45.1, R46.1, R46.2, R47.1, R48.1
- net LINE1_SENSE: now also Q30.1 (G)
- net LINE2_SENSE: now also Q31.1 (G)
- net LINE6_SENSE: now also D19.1 (K), D19.2 (A), Q34.3 (D), Q35.1 (G), R45.2
- new net: D22.1 (K), D22.2 (A), Q37.3 (D), R48.2
- new net: D17.1 (K), D17.2 (A), Q32.3 (D), R43.2
- new net: D20.1 (K), Q35.3 (D)
- new net: D21.2 (A), R47.2
- new net: D16.1 (K), D16.2 (A), Q31.3 (D), R42.2
- new net: D15.1 (K), Q30.3 (D)
- new net: D15.2 (A), R41.2
Other:
- note added: "BSS138 gate on each LINEx_SENSE node (zero DC load: gate leakage <=100nA worst-case = ~5mV on the 47k divider; if one channel ever reads pinned, suspect its Q30-Q37 gate). Drain sinks a super-red 0603 from +3V3 via 1k (~1.4mA). In practice a THRESHOLD indicator: the BSS138's ~150-300mV dark-to-full band makes it crisp on/off around ~1.2V -- ideal for reading line position across 8 LEDs at a glanc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"
- note added: "LINE-SENSOR INDICATORS -- 8 top-side LEDs, one per line channel"

Commit message: Rev 4: WROOM-1 module, 1S power, direct wall ADC, pro routing
User requests: mux only for line array (walls direct to ADC), exact ESP32
library footprint+3D, exact N20 library, speed+RTOS, 1S LiPo, 3 user
buttons, rear USB-C, JTAG outlet, wall indicator LEDs, professional routing.

- ESP32-S3-WROOM-1 (SMD, stock footprint + 3D STEP), antenna overhanging
  the right edge per Espressif rules (interior placement disallowed).
  Locked pin map adversarially verified: JTAG on the real quad IO39-42,
  ENC2 on UART0 pins with 1k boot-contention guards (review blocker),
  straps as idle-low outputs with pull-downs, buttons IO0/35/36.
- 1S LiPo: TPS63001 buck-boost (buck can't hold 3.3V from a sagging cell),
  no balance lead, divider rescaled 4.2V->2.52V (ADC calibrated-range
  review fix), motors on raw cell (3V-wound N20s).
- Sensors: walls direct on ADC1 IO1-6 (fired pair sampled in parallel),
  line array on one CD74HC4067 (HC swap: HEF4067 out of spec at 3.3V),
  emitters ganged in 4 groups (U5 deleted), 6 PMOS wall indicators
  (LED ON = wall seen) + 8 line indicators on top.
- Project-local N20 library (footprint + hand-authored VRML from Pololu
  drawing 0J949); motors placed true-size, keep-outs match real 33mm body.
- Router upgrades: string-pulling post-pass (canonical diagonal+straight
  45-degree geometry, clearance-verified per candidate -- segment count
  halved), two power-width tiers (0.35mm for the SON-pad nets), padded
  slot/hole keep-outs, via-radius-aware keepout test.
- Fixed a real generator bug: loop Z-bend wires shorted nets every 6th
  sensor (netlist audit caught D3/D9 anodes folded into cathode nets) --
  all loop wiring is now straight by construction.

100x114mm, 4 layers, 152 footprints, 1077 tracks / 167 vias, ERC 0,
DRC 0 errors; 12 connections left for GUI finishing (JTAG fan-out, one
USB pair, buck-boost hookup) -- listed in PROJECT_NOTES.

Co-Authored-By: Claude Fable 5 <noreply@anthropic.com>
Parts:
- removed A1: Arduino Nano ESP32 (ESP32-S3) -- sole controller,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, Module:Arduino_Nano, symbol Connector_Generic:Conn_02x15_Odd_Even
- removed C14, C7: 100nF, Capacitor_SMD:C_0805_2012Metric, symbol Device:C
- removed J3: BATT_BALANCE_2S, Connector_JST:JST_XH_B3B-XH-A_1x03_P2.50mm_Vertical, symbol Connector_Generic:Conn_01x03
- removed Q11, Q13, Q15, Q29, Q3, Q30, Q31, Q32, Q33, Q34, Q35, Q36, Q37, Q5, Q7, Q9: BSS138 (real part; Q_NMOS_GSD base symbol used so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, Package_TO_SOT_SMD:SOT-23, symbol Transistor_FET:Q_NMOS_GSD
- removed Q16, Q18, Q20, Q22, Q24, Q26, Q28: SFH309, LED_SMD:LED_1206_3216Metric, symbol Sensor_Optical:SFH309
- removed R4: 10k, Resistor_SMD:R_0805_2012Metric, symbol Device:R
- removed R5: 6.2k, Resistor_SMD:R_0805_2012Metric, symbol Device:R
- removed U1: AP63203WU (fixed 3.3V; symbol is pin-compatible A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, Package_TO_SOT_SMD:TSOT-23-6, symbol Regulator_Switching:AP63200WU
- removed U4, U5: HEF4067BT, Package_SO:SOIC-24W_7.5x15.4mm_P1.27mm, symbol Analog_Switch:HEF4067BT
- added C10: 10uF, Capacitor_SMD:C_0805_2012Metric, symbol Device:C
- added C9: 1uF, Capacitor_SMD:C_0805_2012Metric, symbol Device:C
- added D23, D24, D25, D26, D27, D28: Indicator LED 0603 super-red AlInGaP, high-eff bi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, LED_SMD:LED_0603_1608Metric, symbol LED:LD271
- added J7: USB-C rear (GCT USB4105; VBUS unused -- battery p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, Connector_USB:USB_C_Receptacle_GCT_USB4105-xx-A_16P_TopMnt_Horizontal, symbol Connector:USB_C_Receptacle_USB2.0_16P
- added J8: JTAG_1x6 (3V3,TMS,TCK,TDO,TDI,GND), Connector_PinHeader_2.54mm:PinHeader_1x06_P2.54mm_Vertical, symbol Connector_Generic:Conn_01x06
- added Q11, Q13, Q15, Q9: SFH309, LED_SMD:LED_1206_3216Metric, symbol Sensor_Optical:SFH309
- added Q16, Q18, Q20, Q22, Q24, Q26: BSS138 (real part; Q_NMOS_GSD base symbol used so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, Package_TO_SOT_SMD:SOT-23, symbol Transistor_FET:Q_NMOS_GSD
- added Q28, Q29, Q30, Q31, Q32, Q33: BSS84 (PMOS indicator driver; Q_PMOS base symbol), Package_TO_SOT_SMD:SOT-23, symbol Device:Q_PMOS
- added Q3, Q5, Q7: SFH309, LED_THT:LED_D3.0mm_Clear, symbol Sensor_Optical:SFH309
- added R11, R65, R66: 10k, Resistor_SMD:R_0805_2012Metric, symbol Device:R
- added R12, R56: 5.1k, Resistor_SMD:R_0805_2012Metric, symbol Device:R
- added R49, R50, R51, R52, R53, R54, R57, R58: 1k, Resistor_SMD:R_0805_2012Metric, symbol Device:R
- added R59, R60: 22, Resistor_SMD:R_0805_2012Metric, symbol Device:R
- added R61, R62, R63, R64: 100k, Resistor_SMD:R_0805_2012Metric, symbol Device:R
- added SW2, SW3, SW4: SW_Push, Button_Switch_THT:SW_PUSH_6mm, symbol Switch:SW_Push
- added U1: TPS63001 (fixed 3.3V buck-boost; TPS63000 base sy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, Package_SON:Texas_DRC0010J_ThermalVias, symbol Regulator_Switching:TPS63000
- added U3: ESP32-S3-WROOM-1-N16 (non-R8: octal-PSRAM variant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, RF_Module:ESP32-S3-WROOM-1, symbol RF_Module:ESP32-S3-WROOM-1
- added U4: CD74HC4067M, Package_SO:SOIC-24W_7.5x15.4mm_P1.27mm, symbol 74xx:CD74HC4067M
- added U6: USBLC6-2SC6 (SOT-23-6; 2P6 base symbol so ERC che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, Package_TO_SOT_SMD:SOT-23-6, symbol Power_Protection:USBLC6-2P6
- F1: value 3A_resettable -> 2A_resettable
- J1: value BATT_IN_2S -> BATT_IN_1S; footprint Connector_JST:JST_XH_B2B-XH-A_1x02_P2.50mm_Vertical -> Connector_JST:JST_PH_B2B-PH-K_1x02_P2.00mm_Vertical
- L1: value 3.3uH -> 1.5uH
- Q1: value Q_PMOS (e.g. DMP2035U-7) -> Q_PMOS low-Vth (e.g. DMP2035U-7)
- Q10, Q12, Q8: footprint LED_THT:LED_D3.0mm_Clear -> LED_SMD:LED_1206_3216Metric
- R2: value 10k -> 22k
- R3: value 22k -> 33k
Connections:
- net LINE1_SENSE is gone; now on net GND: Q14.1 (C), R25.2
- net LINE4_LED is gone; now on net GND: Q21.1 (G)
- net LINE5_LED is gone; now on net GND: Q23.1 (G)
- net LINE6_LED is gone; now on net GND: Q25.1 (G)
- net LINE7_LED is gone; now on net GND: Q27.1 (G)
- net VM_BATT is gone; now on net GND: C1.1, C2.1, C4.1, J11.1 (Pin_1), Q1.S
- net AIN1: now also U3.17 (IO9)
- net AIN2: now also U3.18 (IO10)
- net BIN1: now also U3.31 (IO38)
- net BIN2: now also R65.1, U3.26 (IO45)
- net ENC1_A: now also U3.24 (IO47)
- net ENC1_B: now also U3.25 (IO48)
- net ENC2_A: now also R57.1
- net ENC2_B: now also R58.1
- net GND: now also C3.1, C3.2, D1.2 (A), D12.2 (A), D15.2 (A), D16.2 (A), D17.2 (A), D19.2 (A), D2.2 (A), D21.2 (A), D22.2 (A), D3.2 (A), D7.2 (A), D8.2 (A), Q2.1 (C), Q4.1 (C), Q6.1 (C), R13.2, R14.2, R15.2, R16.2, R17.2, R18.2, R2.1, R26.2, R27.2, R28.2, R35.2, R36.2, R41.2, R42.2, R43.2, R45.2, R47.2, R48.2, C10.1, C10.2, C9.2, D23.1 (K), D24.1 (K), D25.1 (K), D26.1 (K), D27.1 (K), D28.1 (K), J7.A1 (GND), J7.A12 (GND), J7.B1 (GND), J7.B12 (GND), J7.SH (SHIELD), J8.1 (Pin_1), J8.6 (Pin_6), Q11.1 (C), Q11.2 (E), Q13.1 (C), Q13.2 (E), Q15.1 (C), Q15.2 (E), Q16.2 (S), Q18.2 (S), Q20.1 (G), Q20.2 (S), Q22.1 (G), Q22.2 (S), Q24.1 (G), Q24.2 (S), Q26.1 (G), Q26.2 (S), Q28.D, Q28.G, Q28.S, Q29.D, Q29.G, Q29.S, Q3.1 (C), Q3.2 (E), Q30.D, Q30.G, Q30.S, Q31.D, Q31.G, Q31.S, Q32.D, Q32.G, Q32.S, Q33.D, Q33.G, Q33.S, Q5.1 (C), Q5.2 (E), Q7.1 (C), Q7.2 (E), Q9.1 (C), Q9.2 (E), R11.1, R12.2, R49.1, R50.1, R51.1, R52.1, R53.1, R54.1, R56.2, R61.2, R62.2, R63.2, R64.2, R65.2, R66.2, SW2.2, SW3.2, SW4.2, U1.1 (VOUT), U1.10 (FB), U1.11 (PGND), U1.3 (PGND), U1.5 (VIN), U1.6 (EN), U1.7 (PS/SYNC), U1.8 (VINA), U1.9 (GND), U3.1 (GND), U3.12 (IO8), U3.15 (IO3), U3.2 (3V3), U3.27 (IO0), U3.38 (IO2), U3.39 (IO1), U3.4 (IO4), U3.40 (GND), U3.41 (GND), U3.5 (IO5), U3.6 (IO6), U4.12 (GND), U4.13 (S3), U4.15 (~{E}), U4.2 (I7), U4.24 (VCC), U4.3 (I6), U4.4 (I5), U4.5 (I4), U4.6 (I3), U4.7 (I2), U4.8 (I1), U4.9 (I0), U6.2 (GND), U6.5 (VBUS); no longer D11.1 (K), D13.1 (K), D18.1 (K), D21.1 (K), D4.1 (K), D5.1 (K), D9.1 (K), L1.2, Q19.3 (D), Q23.3 (D), Q27.3 (D)
- net MUX_S0: now also U3.19 (IO11), U4.10 (S0)
- net MUX_S1: now also U3.20 (IO12), U4.11 (S1)
- net MUX_S2: now also U3.21 (IO13), U4.14 (S2)
- net MUX_SENSE: now also U3.7 (IO7), U4.1 (COM)
- net PWMA: now also U3.11 (IO18)
- net PWMB: now also U3.23 (IO21)
- net STBY: now also R66.1, U3.16 (IO46)
- net EMIT_FRONT_K: now reaches D2.1 (K)
- net EMIT_FRONT_K: now also D1.1 (K), Q16.3 (D)
- net at D20.1 (K): now also Q25.3 (D)
- net EMIT_LINE_K: now reaches D14.1 (K)
- net EMIT_LINE_K: now also D10.1 (K), D11.1 (K), D12.1 (K), D13.1 (K), D7.1 (K), D8.1 (K), D9.1 (K), Q19.3 (D)
- net EMIT_SIDE_K: now reaches D6.1 (K)
- net EMIT_SIDE_K: now also D5.1 (K), Q18.3 (D)
- net at D15.1 (K): now also Q20.3 (D)
- net at Q21.3 (D): now also D16.1 (K); no longer D10.1 (K)
- net at L1.1: now also U1.4 (L1); no longer C3.2
- net LINE2_LED renamed WALL_EMIT_DIAG
- net WALL_EMIT_DIAG: now also R63.1, U3.9 (IO16)
- removed net LINE2_SENSE: D8.1 (K), D8.2 (A), Q17.3 (D), R27.2, R28.2
- net LINE3_LED renamed LINE_EMIT
- net LINE_EMIT: now also R61.1, U3.22 (IO14)
- removed net LINE6_SENSE: D12.1 (K), D12.2 (A), D19.1 (K), D19.2 (A), Q25.3 (D), R35.2, R36.2, R45.2
- removed net WALL1_SENSE: D1.1 (K), D1.2 (A), Q2.1 (C), R13.2, R14.2
- removed net WALL2_SENSE: D2.2 (A), D3.1 (K), D3.2 (A), Q4.1 (C), Q6.1 (C), R15.2, R16.2, R17.2, R18.2
- new net: L1.2, U1.2 (L2)
- new net: D26.2 (A), R52.2
- new net: D27.2 (A), R53.2
- new net: D18.1 (K), Q23.3 (D)
- new net: D19.1 (K), Q24.3 (D)
- new net: D25.2 (A), R51.2
- new net: D24.2 (A), R50.2
- new net: R60.1, U6.4 (I/O2)
- new net: R59.1, U6.6 (I/O1)
- new net: D23.2 (A), R49.2
- new net: D21.1 (K), Q26.3 (D)
- new net: D28.2 (A), R54.2
- new net: J7.A4 (VBUS), J7.A9 (VBUS), J7.B4 (VBUS), J7.B9 (VBUS)
- new net: J7.A5 (CC1), R12.1
- new net: J7.B5 (CC2), R56.1
- new net: D17.1 (K), Q22.3 (D)
- new net: D22.1 (K), Q27.3 (D)
- new net EMIT_DIAG_K: D3.1 (K), D4.1 (K), Q17.3 (D)
- new net ENC2_A_S3: R57.2, U3.36 (RXD0)
- new net ENC2_B_S3: R58.2, U3.37 (TXD0)
- new net ESP_EN: C9.1, R11.2, SW2.1, U3.3 (EN)
- new net JTAG_TCK: J8.3 (Pin_3), U3.32 (IO39)
- new net JTAG_TDI: J8.5 (Pin_5), U3.34 (IO41)
- new net JTAG_TDO: J8.4 (Pin_4), U3.33 (IO40)
- new net JTAG_TMS: J8.2 (Pin_2), U3.35 (IO42)
- new net USB_DM: R59.2, U3.13 (USB_D-)
- new net USB_DM_C: J7.A7 (D-), J7.B7 (D-), U6.1 (I/O1)
- new net USB_DP: R60.2, U3.14 (USB_D+)
- new net USB_DP_C: J7.A6 (D+), J7.B6 (D+), U6.3 (I/O2)
- new net USER_BTN2: SW3.1, U3.28 (IO35)
- new net USER_BTN3: SW4.1, U3.29 (IO36)
- new net WALL_EMIT_FRONT: Q16.1 (G), R62.1, U3.8 (IO15)
- new net WALL_EMIT_SIDE: Q18.1 (G), R64.1, U3.10 (IO17)
- no-connect marks 11 -> 12
Other:
- note added: "+3V3 is the single regulated logic rail: the ESP32-S3 module, mux logic, encoder VCC, phototransistor pull-ups, indicator drivers and IR LED current all come from here."
- note added: "CONTROLLER -- ESP32-S3-WROOM-1 (dual-core 240MHz, FreeRTOS, WiFi): control + telemetry"
- note added: "ESP32-S3-WROOM-1 on FreeRTOS: 6 wall sensors DIRECT on ADC1 IO1-IO6 (a fired pair is sampled in parallel), line array via U4 (IO7 + IO11-13), battery IO8, TB6612 on IO9/10/18/21/38/45/46 (straps 45/46 = idle-low outputs ONLY -- never add pull-ups), encoders IO43/44/47/48 (PCNT hardware quadrature via GPIO matrix), JTAG on the real JTAG quad IO39-42 -> J8 (ESP-Prog). Buttons: SW1=IO0 (start/BOOT),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"
- note added: "ONE HEF4067 (line array only -- user decision 2026-07-15: wall sensors are read directly on ESP32 ADC1 pins). Each sensor: phototransistor (collector -> 47k pull-up to +3V3 AND to its readout node; emitter -> GND) + IR LED (anode -> current-limit resistor -> +3V3; cathode -> its GROUP's low-side switch). Emitters are GANGED: front pair / diagonal pair / side pair / all-8 line bank, each on one BS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"
- note added: "POWER -- 1S LiPo -> TPS63001 buck-boost -> 3V3"
- note added: "SW1 = USER_BTN on IO0: start-run button AND the BOOT strap (hold SW1, tap SW2=reset -> ROM download mode). External 10k pull-up R10 keeps the strap solid. SW3/SW4 = USER_BTN2/3 on IO35/IO36 (menu/select UX): active-low, firmware enables the internal pull-ups -- no external resistors. NOTE: on octal-PSRAM (-R8) modules IO35/36 do not exist; buttons 2/3 are the sacrificial feature (control is unaff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"
- note added: "USER INTERFACE -- 3 buttons"
- note added: "VBAT_SENSE = cell voltage (0-4.2V) scaled to <=2.52V by 22k/33k (the S3 ADC calibrated range tops at ~2.9V with worst error near the top -- keep headroom). Into ADC1 IO8. Firmware low-battery cutoff at 3.0V/cell. Single 1S cell: no balance lead."
- note added: "WALL-SENSOR INDICATORS -- 6 top-side LEDs, LED ON = wall seen (PMOS, inverted node)"
- note removed: "+3V3 is the single regulated logic rail: the ESP32 dev board, mux logic, encoder VCC, phototransistor pull-ups, and IR LED driver current all come from here (not raw VM_BATT)."
- note removed: "2x HEF4067BT 16-ch analog mux/demux, sharing select lines MUX_S0-S3. Each sensor: SFH309 phototransistor (collector -> 47k pull-up to +3V3 AND to its read-mux channel; emitter -> GND) + SFH4550 IR LED (anode -> current-limit resistor -> +3V3; cathode -> BSS138 low-side switch drain; switch source -> GND; switch gate -> its write-demux channel). Firmware pulses LED_PULSE while stepping MUX_S0-S3 t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"
- note removed: "CONNECTORS / DEBUG"
- note removed: "CONTROLLER -- socketed Arduino Nano ESP32 (ESP32-S3): control + sensors + telemetry"
- note removed: "POWER"
- note removed: "Single ESP32-S3 runs everything: TB6612 (STBY/PWMA/PWMB/AIN*/BIN*), 4 encoder inputs, the 2x HEF4067 sensor muxes (MUX_S0-S3 select, MUX_SENSE ADC, LED_PULSE), the two battery-sense ADCs, and USER_BTN. Wi-Fi/BLE telemetry is built in; flashed over the board's own USB-C -- no separate programmer or UART relay. The 3 analog nets are on A0-A2 (real ADC pins). The Nano-ESP32 header-to-GPIO map, and w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"
- note removed: "USER_BTN (ESP32 A7) -- active-low start-run button, pulled up to +3V3. Standard micromouse UX (arm, then start a run). One of the ESP32 analog-capable pins; the full net/pin allocation is in PROJECT_NOTES.md. No separate debug/programming header on this board: the Arduino Nano ESP32 is flashed over its own onboard USB-C, and firmware is updated the same way (or over-the-air via Wi-Fi). No BOOT0/S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"
- note removed: "VBAT_CELL1_SENSE = cell1 voltage (0-4.2V) scaled to <=2.9V. VBAT_PACK_SENSE = full pack voltage (0-8.4V) scaled to <=3.3V. Firmware computes cell2 = pack - cell1. Both wired to ESP32 ADC pins A2/A1 (VBAT_PACK_SENSE/VBAT_CELL1_SENSE) -- see GPIO allocation table in PROJECT_NOTES.md."

Commit message: Rev 5: SMD driver, rear service panel, bracket holes, routed to zero
- TB6612FNG as bare SSOP-24 in the inter-motor corridor; decoupling on B.Cu
- ESP32-S3-WROOM-1 moved to the rear, antenna overhanging the rear edge
  (Espressif-preferred); USB-C, ESD, JTAG and buttons A/B/C (+RST, silk
  letters) grouped around it as a service panel; motors moved forward
- Ø3.2mm/18.0mm-c-c NPTH pairs matching the printable UKMARSBot
  Pololu-pattern N20 bracket (STL link in README/PROJECT_NOTES)
- Wall sensors re-laid per parsed championship practice: detector forward,
  emitter 7.6mm behind, in-line, co-aimed; 10/45/75 degree aims
- USB VBUS turned into a cable-detect divider on IO37 (was a dangling NC)
- Board 100x120mm: +6mm rear fan-out band after routing proved density-bound
- board_geom.py: single source of mechanical truth (placement + router)
- Route-to-zero: jailed-first ordering with immediate retry ladders,
  hand bridges (D+ pair, VBUS stack link on In1), under-body pre-stitch,
  wide verify-proof retry rung, THT-aware clearance floors everywhere,
  all-layer via-replacement stitching, and heal_all.py convergent DRC healer
- Final: 0 unrouted, ERC 0, DRC 0 violations / 0 unconnected / 0 parity

Co-Authored-By: Claude Fable 5 <noreply@anthropic.com>
Parts:
- removed J10: TB6612_BREAKOUT_CTRL, Connector_PinSocket_2.54mm:PinSocket_1x08_P2.54mm_Vertical, symbol Connector_Generic:Conn_01x08
- removed J11: TB6612_BREAKOUT_PWR_OUT, Connector_PinSocket_2.54mm:PinSocket_1x08_P2.54mm_Vertical, symbol Connector_Generic:Conn_01x08
- added C11: 10uF, Capacitor_SMD:C_0805_2012Metric, symbol Device:C
- added C12, C14: 100nF, Capacitor_SMD:C_0805_2012Metric, symbol Device:C
- added R67: 10k, Resistor_SMD:R_0805_2012Metric, symbol Device:R
- added R68: 15k, Resistor_SMD:R_0805_2012Metric, symbol Device:R
- added U2: TB6612FNG, Package_SO:SSOP-24_5.3x8.2mm_P0.65mm, symbol Driver_Motor:TB6612FNG
- SW1: value SW_Push -> BTN_A (start / BOOT)
- SW2: value SW_Push -> RESET
- SW3: value SW_Push -> BTN_B
- SW4: value SW_Push -> BTN_C
Connections:
- net AIN1: now also U2.21 (AIN1)
- net AIN2: now also U2.22 (AIN2)
- net BIN1: now also U2.17 (BIN1)
- net BIN2: now also U2.16 (BIN2)
- net GND: now also C11.1, C11.2, C12.1, C12.2, C14.1, C14.2, R68.2, U2.10 (PGND2), U2.13 (VM2), U2.14 (VM3), U2.18 (GND), U2.20 (VCC), U2.24 (VM1), U2.3 (PGND1), U2.4 (PGND1), U2.9 (PGND2)
- net MOTA_N: now also U2.5 (AO2), U2.6 (AO2)
- net MOTA_P: now also U2.1 (AO1), U2.2 (AO1)
- net MOTB_N: now also U2.7 (BO2), U2.8 (BO2)
- net MOTB_P: now also U2.11 (BO1), U2.12 (BO1)
- net PWMA: now also U2.23 (PWMA)
- net PWMB: now also U2.15 (PWMB)
- net STBY: now also U2.19 (STBY)
- net VBUS_SENSE: now reaches U3.30 (IO37)
- net VBUS_SENSE: now also R67.2, R68.1
- net USB_VBUS: now reaches J7.A4 (VBUS), J7.A9 (VBUS), J7.B4 (VBUS), J7.B9 (VBUS)
- net USB_VBUS: now also R67.1
- no-connect marks 12 -> 10
Other:
- note added: "Bare TB6612FNG (U2, SSOP-24): STBY/AIN/BIN plain GPIO, PWMA/PWMB = LEDC. VM = raw 1S cell (2.5V min OK), VCC = +3V3. Doubled pins (AO1/AO2/BO1/BO2 pairs, PGND pairs, VM triple) are bridged by the router's micro-bridge pass. Decoupling at the chip: C11 10uF + C12 100nF on VM, C14 100nF on VCC."
- note added: "Buttons are lettered on the silkscreen: A=SW1, B=SW3, C=SW4, RST=SW2. SW1/A = USER_BTN on IO0: start-run button AND the BOOT strap (hold A, tap RST -> ROM download mode). External 10k pull-up R10 keeps the strap solid. SW3/SW4 = USER_BTN2/3 on IO35/IO36 (menu/select UX): active-low, firmware enables the internal pull-ups -- no external resistors. NOTE: on octal-PSRAM (-R8) modules IO35/36 do not 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"
- note added: "MOTOR DRIVER (TB6612FNG, SMD) -- 2x N20-with-encoder motors"
- note removed: "Breakout logic inputs: STBY, AIN1/AIN2, BIN1/BIN2 are plain ESP32 GPIO; PWMA/PWMB are ESP32 LEDC PWM outputs (firmware configures PWM). VM=raw battery, VCC=+3V3 logic, GND common. AO1/AO2 -> motor A (MOTA_P/N), BO1/BO2 -> motor B (MOTB_P/N). The breakout's own board carries VM/VCC decoupling. VERIFY the breakout's real pin order + row spacing before fab."
- note removed: "MOTOR DRIVER (socketed TB6612 breakout) + ENCODERS -- 2x N20-with-encoder motors"
- note removed: "SW1 = USER_BTN on IO0: start-run button AND the BOOT strap (hold SW1, tap SW2=reset -> ROM download mode). External 10k pull-up R10 keeps the strap solid. SW3/SW4 = USER_BTN2/3 on IO35/IO36 (menu/select UX): active-low, firmware enables the internal pull-ups -- no external resistors. NOTE: on octal-PSRAM (-R8) modules IO35/36 do not exist; buttons 2/3 are the sacrificial feature (control is unaff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"
