File: pcb/micromouse-pcb.kicad_sch (KiCad schematic)
At the start: 156 parts, among them J1 BATT_IN_1S, J2 EXT_SWITCH, J5 MOTOR_A_N20_ENCODER, J6 MOTOR_B_N20_ENCODER, J7 USB-C rear (GCT USB4105; VBUS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, J8 JTAG_1x6 (3V3,TMS,TCK,TDO,TDI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, Q1 Q_PMOS low-Vth (e.g. DMP2035U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, Q10 SFH309, Q11 SFH309, Q12 SFH309, Q13 SFH309, Q14 SFH309, Q15 SFH309, Q16 BSS138 (real part; Q_NMOS_GSD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, Q17 BSS138 (real part; Q_NMOS_GSD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, Q18 BSS138 (real part; Q_NMOS_GSD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, Q19 BSS138 (real part; Q_NMOS_GSD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, Q2 SFH309, Q20 BSS138 (real part; Q_NMOS_GSD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, Q21 BSS138 (real part; Q_NMOS_GSD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, Q22 BSS138 (real part; Q_NMOS_GSD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, Q23 BSS138 (real part; Q_NMOS_GSD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, Q24 BSS138 (real part; Q_NMOS_GSD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, Q25 BSS138 (real part; Q_NMOS_GSD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, Q26 BSS138 (real part; Q_NMOS_GSD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, Q27 BSS138 (real part; Q_NMOS_GSD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, Q28 BSS84 (PMOS indicator driver;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, Q29 BSS84 (PMOS indicator driver;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, Q3 SFH309, Q30 BSS84 (PMOS indicator driver;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, Q31 BSS84 (PMOS indicator driver;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, Q32 BSS84 (PMOS indicator driver;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, Q33 BSS84 (PMOS indicator driver;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, Q4 SFH309, Q5 SFH309, Q6 SFH309, Q7 SFH309, Q8 SFH309, Q9 SFH309, SW1 BTN_A (start / BOOT), SW2 RESET, SW3 BTN_B, SW4 BTN_C, U1 TPS63001 (fixed 3.3V buck-boo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, U2 TB6612FNG, U3 ESP32-S3-WROOM-1-N16 (non-R8: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, U4 CD74HC4067M, U6 USBLC6-2SC6 (SOT-23-6; 2P6 ba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

Commit message: Rev 5.1: fix floating FETs (audit-caught), NPTH bracket holes, hard gates
An adversarial audit of shipped rev 5 found Q1 + Q28-Q33 electrically
floating: Device:Q_PMOS numbers its pins D/G/S, the SOT-23 pads are 1/2/3,
and PcbGen silently skipped unmatched pads -- netless pads make no ratsnest,
so both the router and DRC connectivity were structurally blind. The battery
power path (J2 -> F1 -> Q1 -> VM_BATT) was open and all six wall-indicator
drivers were dead. Full postmortem in PROJECT_NOTES.md.

- QPMOS now instantiates Transistor_FET:Q_PMOS_GSD (pins 1/2/3, same
  geometry); netlist verified pin-by-pin, board rerouted to zero
- NEW hard gate: PcbGen.assert_netlist_pads_mapped() in build_pcb.py --
  every netlist (ref,pin) must exist as a board pad carrying that net
- net_conflict parity severity raised warning -> error in .kicad_pro
- verify_netlist.py rewritten for rev-5 topology (was rev-1 names, always
  exit 0); now checks the battery path and sensor->reader->indicator
  reachability, exits 1 on failure
- Mounting holes converted from Edge.Cuts circles to real NPTH pads
  (H1-H5, board-only footprints): drilled, in the fab hole table, matching
  the documented "Ø3.2mm NPTH" claim; keepouts now admit footprint pads
- heal_all.py: no more stacked bridge vias on unfixable fragments
- Docs: U3 anchor corrected to (35.25,113.5); stale rev-3/4 renders removed
- Verified: ERC 0 | DRC 0 violations / 0 unconnected / 0 parity (with
  net_conflict at error severity) | verify_netlist PASSES | 454/454 pins
  mapped | Q1 pads on Net-(Q1-G)/VM_BATT/Net-(Q1-D) with routed copper

Co-Authored-By: Claude Fable 5 <noreply@anthropic.com>
Parts:
- removed Q1: Q_PMOS low-Vth (e.g. DMP2035U-7), Package_TO_SOT_SMD:SOT-23, symbol Device:Q_PMOS
- removed Q28, Q29, Q30, Q31, Q32, Q33: BSS84 (PMOS indicator driver; Q_PMOS base symbol), Package_TO_SOT_SMD:SOT-23, symbol Device:Q_PMOS
- added Q1: Q_PMOS low-Vth (e.g. DMP2035U-7), Package_TO_SOT_SMD:SOT-23, symbol Transistor_FET:Q_PMOS_GSD
- added Q28, Q29, Q30, Q31, Q32, Q33: BSS84 (PMOS indicator driver; Q_PMOS base symbol), Package_TO_SOT_SMD:SOT-23, symbol Transistor_FET:Q_PMOS_GSD
Connections:
- net GND: now also Q1.2 (S), Q28.1 (G), Q28.2 (S), Q28.3 (D), Q29.1 (G), Q29.2 (S), Q29.3 (D), Q30.1 (G), Q30.2 (S), Q30.3 (D), Q31.1 (G), Q31.2 (S), Q31.3 (D), Q32.1 (G), Q32.2 (S), Q32.3 (D), Q33.1 (G), Q33.2 (S), Q33.3 (D)
- net at F1.2: now also Q1.3 (D)
- net at R1.1: now also Q1.1 (G)

Commit message: Rev 5.2: verified-MPN BOM, complete STEP coverage, gated fab exports
Closes the three deferred audit items:

- BOM.csv: 42 line items, 100% MPN coverage. Every part adversarially
  verified against datasheets + live distributor stock (31 parts, two
  research passes): packages vs footprints, SOT-23 FET pinouts (1=G/2=S/3=D).
  Catches: USBLC6-2P6 would have been the wrong package (SOT-666) -> 2SC6;
  module pinned to -N16 (octal-PSRAM variants consume IO35-37 which this
  design uses); L1 -> SRP7028A-1R5M (datasheet-typical 1.5uH, verified
  orderable); line array = IR11-21C/TR8 + PT11-21B/L41/TR8 (true 1206,
  daylight-filtered PT required). SOURCING ALARM: SFH 309 FA is Last Time
  Buy 2026-12-01.
- MPN/Manufacturer emitted as hidden schematic fields via a gen_sch
  field_provider; fixed latent value-plumbing bug (photo_val/led_val never
  passed -- SMD line parts were VALUE-labeled as THT parts); 147 board
  Value fields re-synced; net topology proven byte-identical.
- gen_step_models.py: hand-authored AP214 box-solid STEP for the N20 motors
  and for U1/L1 (KiCad ships no models for those footprints); U1/L1
  repointed to project-local models (text-level -- pcbnew Models() is a
  SWIG copy); STEP export now loads EVERY model.
- export_fab.py: gerbers/drill/pos/STEP/BOM with hard gates (3.2+3.0mm NPTH
  tools must be in the drill data, no missing 3D models, all layers
  non-trivial, BOM MPN coverage reported). ALL GATES PASSED.
- Final state unchanged and re-verified: ERC 0, DRC 0/0/0, netlist gate
  passes.

Co-Authored-By: Claude Fable 5 <noreply@anthropic.com>
Parts:
- C1: MPN (none) -> CL32A107MQVNNNE; Manufacturer (none) -> Samsung Electro-Mechanics
- C10, C11, C4: MPN (none) -> CL21A106KPFNNNE; Manufacturer (none) -> Samsung Electro-Mechanics
- C12, C13, C14, C2, C3, C6, C8: MPN (none) -> CL21B104KBCNNNC; Manufacturer (none) -> Samsung Electro-Mechanics
- C5: MPN (none) -> CL21A226KPCLRNC; Manufacturer (none) -> Samsung Electro-Mechanics
- C9: MPN (none) -> CL21B105KAFNNNE; Manufacturer (none) -> Samsung Electro-Mechanics
- D1, D2, D3, D4, D5, D6: value SFH4550 (real part; LD271 base symbol used so ERC checks pins) -> SFH4550 (THT, LD271 base symbol); MPN (none) -> SFH 4550; Manufacturer (none) -> ams-OSRAM
- D10, D11, D12, D13, D14, D7, D8, D9: value SFH4550 (real part; LD271 base symbol used so ERC checks pins) -> IR11-21C 940nm 1206 IR emitter (LD271 sym for ERC); MPN (none) -> IR11-21C/TR8; Manufacturer (none) -> Everlight
- D15, D16, D17, D18, D19, D20, D21, D22, D23, D24, D25, D26, D27, D28: MPN (none) -> APT1608SURCK; Manufacturer (none) -> Kingbright
- F1: MPN (none) -> 0ZCJ0200FF2C; Manufacturer (none) -> Bel Fuse
- J1: MPN (none) -> B2B-PH-K-S(LF)(SN); Manufacturer (none) -> JST
- J2: MPN (none) -> 61300211121; Manufacturer (none) -> Wurth Elektronik
- J5, J6: MPN (none) -> B6B-PH-K-S(LF)(SN); Manufacturer (none) -> JST
- J7: MPN (none) -> USB4105-GF-A; Manufacturer (none) -> GCT
- J8: MPN (none) -> 61300611121; Manufacturer (none) -> Wurth Elektronik
- L1: MPN (none) -> SRP7028A-1R5M; Manufacturer (none) -> Bourns
- Q1: MPN (none) -> DMP2035U-7; Manufacturer (none) -> Diodes Incorporated
- Q10, Q11, Q12, Q13, Q14, Q15, Q8, Q9: value SFH309 -> PT11-21B/L41 940nm 1206 phototransistor, DAYLIGHT-FILTERED (black lens) REQUIRED -- an unfiltered part (PT11-21C) re-op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; MPN (none) -> PT11-21B/L41/TR8; Manufacturer (none) -> Everlight
- Q16, Q17, Q18, Q19, Q20, Q21, Q22, Q23, Q24, Q25, Q26, Q27: MPN (none) -> BSS138LT1G; Manufacturer (none) -> onsemi
- Q2, Q3, Q4, Q5, Q6, Q7: MPN (none) -> SFH 309 FA; Manufacturer (none) -> ams-OSRAM
- Q28, Q29, Q30, Q31, Q32, Q33: MPN (none) -> BSS84LT1G; Manufacturer (none) -> onsemi
- R1, R61, R62, R63, R64: MPN (none) -> RC0805FR-07100KL; Manufacturer (none) -> Yageo
- R10, R11, R6, R65, R66, R67, R7, R8, R9: MPN (none) -> RC0805FR-0710KL; Manufacturer (none) -> Yageo
- R12, R56: MPN (none) -> RC0805FR-075K1L; Manufacturer (none) -> Yageo
- R13, R15, R17, R19, R21, R23, R25, R27, R29, R31, R33, R35, R37, R39: MPN (none) -> RC0805FR-0747KL; Manufacturer (none) -> Yageo
- R14, R16, R18, R20, R22, R24: MPN (none) -> RC0805FR-0733RL; Manufacturer (none) -> Yageo
- R2: MPN (none) -> RC0805FR-0722KL; Manufacturer (none) -> Yageo
- R26, R28, R30, R32, R34, R36, R38, R40: MPN (none) -> RC0805FR-07120RL; Manufacturer (none) -> Yageo
- R3: MPN (none) -> RC0805FR-0733KL; Manufacturer (none) -> Yageo
- R41, R42, R43, R44, R45, R46, R47, R48, R49, R50, R51, R52, R53, R54, R57, R58: MPN (none) -> RC0805FR-071KL; Manufacturer (none) -> Yageo
- R59, R60: MPN (none) -> RC0805FR-0722RL; Manufacturer (none) -> Yageo
- R68: MPN (none) -> RC0805FR-0715KL; Manufacturer (none) -> Yageo
- SW1, SW2, SW3, SW4: MPN (none) -> B3F-1000; Manufacturer (none) -> Omron
- U1: MPN (none) -> TPS63001DRCR; Manufacturer (none) -> Texas Instruments
- U2: MPN (none) -> TB6612FNG,C,8,EL; Manufacturer (none) -> Toshiba
- U3: MPN (none) -> ESP32-S3-WROOM-1-N16; Manufacturer (none) -> Espressif Systems
- U4: MPN (none) -> CD74HC4067M96; Manufacturer (none) -> Texas Instruments
- U6: MPN (none) -> USBLC6-2SC6; Manufacturer (none) -> STMicroelectronics

Commit message: Rev 5.3: routed to zero, wire-level verification, firmware + host sim
Board: rear-facing USB-C, soft EN switch (SW5), JTAG at rear, per-sensor
wall indicator LEDs, inboard bent-lead wall optics with silkscreen body
outlines, open edge wheel notches, India-available optos (TCRT5000 line,
PT334-6B wall). DRC 0 violations / 0 unconnected / 0 parity; ERC 0.

Verification: 28/28 netlist-computed circuit tests (TEST_REPORT.md),
trace-level copper analysis with pad-junction/T-split graph physics
(TRACE_REPORT.md), 30 firmware pins gated against the netlist, host sim
of the shipped control core passes all scenarios (caught 2 real control
bugs pre-hardware). Fab gates ALL PASSED; 42-line verified-MPN BOM.

Firmware: fw/micromouse (pins.h, control core, .ino with LEDC/PCNT/mux
scan/pulsed emitters), fw/sim host simulation, fw/check_pins.py gate.

Co-Authored-By: Claude Fable 5 <noreply@anthropic.com>
Parts:
- removed D10, D11, D12, D13, D14, D7, D8, D9: IR11-21C 940nm 1206 IR emitter (LD271 sym for ERC), LED_SMD:LED_1206_3216Metric, symbol LED:LD271
- removed J2: EXT_SWITCH, Connector_PinHeader_2.54mm:PinHeader_1x02_P2.54mm_Vertical, symbol Connector_Generic:Conn_01x02
- removed Q10, Q11, Q12, Q13, Q14, Q15, Q8, Q9: PT11-21B/L41 940nm 1206 phototransistor, DAYLIGHT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, LED_SMD:LED_1206_3216Metric, symbol Sensor_Optical:SFH309
- added LS1, LS2, LS3, LS4, LS5, LS6, LS7, LS8: TCRT5000 (reflective sensor, filtered PT; PC817 b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, n20:TCRT5000, symbol Isolator:PC817
- added R69: 1M, Resistor_SMD:R_0805_2012Metric, symbol Device:R
- added SW5: PWR (OS102011MS2QN1 slide; slide-to-GND = OFF), Button_Switch_THT:SW_Slide_SPDT_Straight_CK_OS102011MS2Q, symbol Switch:SW_SPDT
- D1, D2, D3, D4, D5, D6: value SFH4550 (THT, LD271 base symbol) -> SFH4550 (THT, LD271 base symbol; India alternate: TSAL6100)
- Q2, Q3, Q4, Q5, Q6, Q7: value SFH309 -> PT334-6B (5mm filtered PT; LONG LEAD = EMITTER; SFH309 base symbol so ERC checks pins); footprint LED_THT:LED_D3.0mm_Clear -> LED_THT:LED_D5.0mm_IRBlack; MPN SFH 309 FA -> PT334-6B; Manufacturer ams-OSRAM -> Everlight
Connections:
- net EMIT_LINE_K is gone; now on net GND: Q19.3 (D)
- net GND: now also LS1.1, LS1.2, LS1.3, LS1.4, LS2.1, LS2.2, LS2.3, LS2.4, LS3.1, LS3.2, LS3.3, LS3.4, LS4.1, LS4.2, LS4.3, LS4.4, LS5.1, LS5.2, LS5.3, LS5.4, LS6.1, LS6.2, LS6.3, LS6.4, LS7.1, LS7.2, LS7.3, LS7.4, LS8.1, LS8.2, LS8.3, LS8.4, R69.1, SW5.1 (A); no longer U1.6 (EN)
- net at J1.1 (Pin_1): now also F1.1
- new net PWR_EN: R69.2, SW5.2 (B), U1.6 (EN)
- no-connect marks 10 -> 11

Commit message: Rev 6.1: 2S power, regulated 6V motors, BNO055 IMU, dual switches + full handoff
Design + firmware + verification COMPLETE and passing; PCB routed to 5
remaining unconnected edges (all in the USB-C connector fanout + the Q1 gate,
documented exactly in HANDOFF.md). This commit is a self-contained handoff so
the board can be finished on another machine with no human input.

Rev 6 (all 10 user requirements, each gated):
- 2S LiPo -> AP63203 3.3V + TPS54302 regulated 6.0V motor rail; DMP3098L
  reverse-FET (Vgs +/-20V, 2S-safe); dual switches (SW5 all / SW6 motors).
- BNO055 9-axis IMU on the centerline (I2C); external crystal DROPPED
  (internal oscillator, spec-supported) after it proved unroutable at the
  0.5mm-pitch LGA.
- Exact wall-sensor aims 0/45/90 deg with silk angle callouts; sensor
  outlines fully inside the board with a 3-5mm edge gap.
- Antenna spans a rear-edge U-notch (nothing outside the outline but shafts).
- USB-C direct D+/D-, IN/IN motor drive, per-cell battery monitoring.
- BOM entirely from Lion Circuits in-stock parts (turnkey, not LCSC).

circuit_tests 41/41 PASS (100% net + component coverage) and CAUGHT A REAL
BUG: the motor rail could never enable (R69 1M source impedance sagged the EN
divider below threshold) -- fixed R69->100k, R70->220k. ERC 0, netlist verify
PASS, 29 firmware pins gated, host sim ALL SCENARIOS PASS.

New tooling: finalize.py (silk->fab + RATSNEST-GATED copper cleanup),
sync_board_meta.py (board<->schematic parity metadata), gen_rev6_libs.py
(BNO055 + SRP4020TA footprints). Key lesson documented: kicad-cli's headless
"unconnected" is unreliable -- the pcbnew ratsnest is the connectivity truth,
and finalize refuses to strip unless it is already zero.

See HANDOFF.md for the exact remaining work, coordinates, gotchas (SWIG traps,
the connectivity trap), and the full finish + regenerate sequences.
Co-Authored-By: Claude Fable 5 <noreply@anthropic.com>
Parts:
- removed R59, R60: 22, Resistor_SMD:R_0805_2012Metric, symbol Device:R
- removed R66: 10k, Resistor_SMD:R_0805_2012Metric, symbol Device:R
- removed U1: TPS63001 (fixed 3.3V buck-boost; TPS63000 base sy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, Package_SON:Texas_DRC0010J_ThermalVias, symbol Regulator_Switching:TPS63000
- added C15, C19, C20, C23: 100nF, Capacitor_SMD:C_0805_2012Metric, symbol Device:C
- added C16, C17: 22uF/25V, Capacitor_SMD:C_1210_3225Metric, symbol Device:C
- added C18: 10uF/25V, Capacitor_SMD:C_1210_3225Metric, symbol Device:C
- added C24: 10uF, Capacitor_SMD:C_0805_2012Metric, symbol Device:C
- added C30: 220uF/16V, Capacitor_SMD:CP_Elec_6.3x7.7, symbol Device:C
- added C7: 22uF, Capacitor_SMD:C_0805_2012Metric, symbol Device:C
- added J9: BALANCE_2S, Connector_JST:JST_XH_B3B-XH-A_1x03_P2.50mm_Vertical, symbol Connector_Generic:Conn_01x03
- added L2: 4.7uH, n20:L_Bourns_SRP4020TA, symbol Device:L
- added R55, R79, R80: 10k, Resistor_SMD:R_0805_2012Metric, symbol Device:R
- added R70: 220k, Resistor_SMD:R_0805_2012Metric, symbol Device:R
- added R71: 110k, Resistor_SMD:R_0805_2012Metric, symbol Device:R
- added R73, R75, R76: 100k, Resistor_SMD:R_0805_2012Metric, symbol Device:R
- added R74: 11k, Resistor_SMD:R_0805_2012Metric, symbol Device:R
- added R77, R78: 4.7k, Resistor_SMD:R_0805_2012Metric, symbol Device:R
- added SW6: PWR MOTORS (PCM12SMTR slide; slide-to-GND = motor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, Button_Switch_SMD:SW_SPDT_PCM12, symbol Switch:SW_SPDT
- added U1: AP63203WU-7 (fixed 3.3V 2A buck; AP63200WU base s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, Package_TO_SOT_SMD:TSOT-23-6, symbol Regulator_Switching:AP63200WU
- added U7: TPS54302DDCR (6.0V/3A motor buck; FB=100k/11k), Package_TO_SOT_SMD:SOT-23-6, symbol Regulator_Switching:TPS54302
- added U8: BNO055 (9-axis IMU + fusion; 3.3V native; I2C 0x2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, n20:BNO055, symbol Sensor_Motion:BNO055
- C1: value 100uF -> 10uF/25V; MPN CL32A107MQVNNNE -> CL32B106KBJNNNE
- C11, C4: value 10uF -> 10uF/25V; footprint Capacitor_SMD:C_0805_2012Metric -> Capacitor_SMD:C_1210_3225Metric; MPN CL21A106KPFNNNE -> CL32B106KBJNNNE
- D1, D2, D3, D4, D5, D6: value SFH4550 (THT, LD271 base symbol; India alternate: TSAL6100) -> IR333-A (Everlight 5mm 940nm 20deg; LD271 base symbol; TSAL6400 is lifecycle-Obsolete at Lion); MPN SFH 4550 -> IR333-A; Manufacturer ams-OSRAM -> Everlight
- F1: value 2A_resettable -> 2.6A/16V PPTC; footprint Fuse:Fuse_1206_3216Metric -> Fuse:Fuse_1812_4532Metric; MPN 0ZCJ0200FF2C -> MINISMDC260F/16-2; Manufacturer Bel Fuse -> Littelfuse
- J1: value BATT_IN_1S -> BATT_IN_2S; footprint Connector_JST:JST_PH_B2B-PH-K_1x02_P2.00mm_Vertical -> Connector_JST:JST_XH_B2B-XH-A_1x02_P2.50mm_Vertical; MPN B2B-PH-K-S(LF)(SN) -> B2B-XH-A
- L1: value 1.5uH -> 4.7uH; footprint Inductor_SMD:L_Bourns_SRP7028A_7.3x6.6mm -> n20:L_Bourns_SRP4020TA; MPN SRP7028A-1R5M -> SRP4020TA-4R7M
- Q1: value Q_PMOS low-Vth (e.g. DMP2035U-7) -> Q_PMOS reverse guard (DMP3098L-7: Vgs +/-20V, 2S-safe); MPN DMP2035U-7 -> DMP3098L-7
- R2: value 22k -> 100k; MPN RC0805FR-0722KL -> RC0805FR-07100KL
- R3: value 33k -> 39k; MPN RC0805FR-0733KL -> RC0805FR-0739KL
- R69: value 1M -> 100k; MPN RC0805FR-071ML -> RC0805FR-07100KL
- SW1, SW2, SW3, SW4: MPN B3F-1000 -> PTS645VL582LFS; Manufacturer Omron -> C&K
- SW5: value PWR (OS102011MS2QN1 slide; slide-to-GND = OFF) -> PWR ALL (PCM12SMTR slide; slide-to-GND = OFF); footprint Button_Switch_THT:SW_Slide_SPDT_Straight_CK_OS102011MS2Q -> Button_Switch_SMD:SW_SPDT_PCM12; MPN OS102011MS2QN1 -> PCM12SMTR
- U3: value ESP32-S3-WROOM-1-N16 (non-R8: octal-PSRAM variants lose IO35-37 = buttons 2/3) -> ESP32-S3-WROOM-1-N8R2 (quad PSRAM: IO35-37 usable; octal -R8 would lose them); MPN ESP32-S3-WROOM-1-N16 -> ESP32-S3-WROOM-1-N8R2
Connections:
- net PWR_EN is gone; now on net ENC2_A: R69.2, SW5.2 (B)
- net ENC2_A: now also R70.1, R70.2, R71.1, SW6.2 (B), U1.2 (EN), U7.5 (EN)
- net GND: now also L1.2, U2.15 (PWMB), U2.23 (PWMA), U4.22 (I9), U4.23 (I8), C16.2, C17.2, C18.1, C18.2, C19.1, C19.2, C20.2, C23.1, C23.2, C24.1, C24.2, C30.2, C7.1, C7.2, J9.1 (Pin_1), J9.2 (Pin_2), R55.1, R71.2, R74.2, R75.1, R75.2, R76.1, R76.2, R77.1, R78.1, R79.1, R80.1, SW6.1 (A), U1.1 (FB), U1.3 (IN), U1.4 (GND), U7.1 (GND), U7.3 (VIN), U8.17 (COM3), U8.18 (COM2), U8.2 (GND), U8.25 (GNDIO), U8.28 (VDDIO), U8.3 (VDD), U8.5 (PS1), U8.6 (PS0); no longer C11.1, C12.1, C3.1, C3.2, U2.13 (VM2), U2.14 (VM3), U2.24 (VM1), U3.12 (IO8), U4.13 (S3)
- net USB_DM: now also U6.6 (I/O1)
- net USB_DP: now also U6.4 (I/O2)
- net VBUS_SENSE: now also U4.21 (I10); no longer U3.30 (IO37)
- net SW_3V3: now reaches L1.1
- net SW_3V3: now also C3.1, C3.2, U1.5 (SW), U1.6 (BST)
- net BATT_RAW: now reaches F1.1, J1.1 (Pin_1)
- net BATT_RAW: now also J9.3 (Pin_3)
- net PWMA renamed IMU_SDA
- net IMU_SDA: now also R77.2, U8.20 (COM0); no longer U2.23 (PWMA)
- net PWMB renamed IMU_SCL
- net IMU_SCL: now also R78.2, U8.19 (COM1); no longer U2.15 (PWMB)
- net STBY: no longer names the net of U2.19 (STBY)
- net STBY: now also R55.2; no longer U3.16 (IO46)
- new net: R79.2, R80.2, U8.11 (~{RESET}), U8.4 (~{BOOT_LOAD_PIN})
- new net: C20.1, U8.9 (CAP)
- new net: C15.2, U7.6 (BOOT)
- new net FB_6V: R73.2, R74.1, U7.4 (FB)
- new net IMU_INT: U3.30 (IO37), U8.14 (INT)
- new net MUX_S3: U3.12 (IO8), U4.13 (S3)
- new net SW_6V: C15.1, L2.1, U7.2 (SW)
- new net VM_6V: C11.1, C12.1, C16.1, C17.1, C30.1, L2.2, R73.1, U2.13 (VM2), U2.14 (VM3), U2.24 (VM1)
- no-connect marks 11 -> 13
Other:
- note added: "+3V3 is the regulated logic rail: ESP32-S3, mux, IMU, encoder VCC, PT pull-ups, indicator drivers and IR LED current. VM_6V feeds ONLY the TB6612 VM pins."
- note added: "BNO055 mid-line placement (user requirement): geometric center of rotation sensing. Mag data is calibration-grade only on a motor robot (1A at 5mm ~ Earth field); the yaw-rate loop uses the gyro. Fusion runs on-chip (100Hz NDOF) or raw gyro at 523Hz."
- note added: "Bare TB6612FNG (U2, SSOP-24) in IN/IN PWM mode: PWMA/PWMB tied 3V3, AIN/BIN = LEDC (IN1=PWM,IN2=0 fwd-coast; IN1=PWM,IN2=1 rev-brake). VM = regulated 6.0V rail (TPS54302, 3A limit) gated by SW6; STBY pulled high (R55) -- motor kill = SW6 + IN pins' internal pull-downs. Decoupling: C30 220uF/16V alu + C11 10uF/25V + C12 100nF on VM, C14 on VCC."
- note added: "IMU -- BNO055 9-axis on I2C (IO18=SDA, IO21=SCL, IO37=INT), addr 0x28; internal osc"
- note added: "POWER -- 2S LiPo -> AP63203 3V3 (2A) + TPS54302 6V motor rail (3A); SW5=logic, SW6=motors"
- note added: "VBAT_SENSE = pack (0-8.4V) x 39/139 <= 2.36V; BAT_MID_SENSE = cell-1 (0-4.2V) x 1/2 <= 2.1V. Both + VBUS_SENSE read through mux channels Y8/Y9/Y10 (ADC1 IO7). Firmware cutoff: 3.3V/cell (either cell) = 6.6V pack floor; the 6V rail is in regulation across that window."
- note removed: "+3V3 is the single regulated logic rail: the ESP32-S3 module, mux logic, encoder VCC, phototransistor pull-ups, indicator drivers and IR LED current all come from here."
- note removed: "Bare TB6612FNG (U2, SSOP-24): STBY/AIN/BIN plain GPIO, PWMA/PWMB = LEDC. VM = raw 1S cell (2.5V min OK), VCC = +3V3. Doubled pins (AO1/AO2/BO1/BO2 pairs, PGND pairs, VM triple) are bridged by the router's micro-bridge pass. Decoupling at the chip: C11 10uF + C12 100nF on VM, C14 100nF on VCC."
- note removed: "POWER -- 1S LiPo -> TPS63001 buck-boost -> 3V3"
- note removed: "VBAT_SENSE = cell voltage (0-4.2V) scaled to <=2.52V by 22k/33k (the S3 ADC calibrated range tops at ~2.9V with worst error near the top -- keep headroom). Into ADC1 IO8. Firmware low-battery cutoff at 3.0V/cell. Single 1S cell: no balance lead."
