File: pcb/micromouse-pcb.kicad_sch (KiCad schematic)
At the start: 172 parts, among them J1 BATT_IN_2S, J5 MOTOR_A_N20_ENCODER, J6 MOTOR_B_N20_ENCODER, J7 USB-C rear (GCT USB4105; VBUS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, J8 JTAG_1x6 (3V3,TMS,TCK,TDO,TDI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, J9 BALANCE_2S, Q1 Q_PMOS reverse guard (DMP3098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, Q16 BSS138 (real part; Q_NMOS_GSD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, Q17 BSS138 (real part; Q_NMOS_GSD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, Q18 BSS138 (real part; Q_NMOS_GSD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, Q19 BSS138 (real part; Q_NMOS_GSD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, Q2 PT334-6B (5mm filtered PT; LO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, Q20 BSS138 (real part; Q_NMOS_GSD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, Q21 BSS138 (real part; Q_NMOS_GSD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, Q22 BSS138 (real part; Q_NMOS_GSD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, Q23 BSS138 (real part; Q_NMOS_GSD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, Q24 BSS138 (real part; Q_NMOS_GSD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, Q25 BSS138 (real part; Q_NMOS_GSD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, Q26 BSS138 (real part; Q_NMOS_GSD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, Q27 BSS138 (real part; Q_NMOS_GSD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, Q28 BSS84 (PMOS indicator driver;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, Q29 BSS84 (PMOS indicator driver;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, Q3 PT334-6B (5mm filtered PT; LO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, Q30 BSS84 (PMOS indicator driver;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, Q31 BSS84 (PMOS indicator driver;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, Q32 BSS84 (PMOS indicator driver;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, Q33 BSS84 (PMOS indicator driver;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, Q4 PT334-6B (5mm filtered PT; LO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, Q5 PT334-6B (5mm filtered PT; LO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, Q6 PT334-6B (5mm filtered PT; LO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, Q7 PT334-6B (5mm filtered PT; LO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, SW1 BTN_A (start / BOOT), SW2 RESET, SW3 BTN_B, SW4 BTN_C, SW5 PWR ALL (PCM12SMTR slide; sli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, SW6 PWR MOTORS (PCM12SMTR slide; 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, U1 AP63203WU-7 (fixed 3.3V 2A bu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, U2 TB6612FNG, U3 ESP32-S3-WROOM-1-N8R2 (quad P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, U4 CD74HC4067M, U6 USBLC6-2SC6 (SOT-23-6; 2P6 ba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, U7 TPS54302DDCR (6.0V/3A motor b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, U8 BNO055 (9-axis IMU + fusion; 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

Commit message: BOM: every part verified In-Stock at Lion; swap OOS motor connector to B6B-XH-A
Individually verified all 43 BOM MPNs against lioncircuits.com. 42 are In
Stock; the only Out-of-Stock part was the motor connector B6B-PH-K-S(LF)(SN)
(the whole top-entry THT JST-PH line is un-stocked at Lion). Swapped J5/J6 to
B6B-XH-A (JST-XH, In Stock, top-entry THT, 2.5mm pitch -- more robust for the
~1.6A motor-stall current).

The XH connector is wider than the 2.0mm PH, so J5/J6 were relocated
(J5->(33,72.5), J6->(83,64), both verified clear of the motor courtyards) and
the board is being rerouted (the previous route was for the PH pad pitch).
This commit has the updated schematic (ERC 0, netlist verify PASS), the
regenerated BOM (B6B-XH-A, no PH parts), build_pcb placement, and the freshly
placed (pre-reroute) board. HANDOFF.md 4a lists the full per-part verification.

All resistors (13 Yageo values), caps (6 Samsung), FETs, LED, and the Wurth
JTAG header confirmed In Stock with dedicated Lion pages.

Co-Authored-By: Claude Fable 5 <noreply@anthropic.com>
Parts:
- J5, J6: footprint Connector_JST:JST_PH_B6B-PH-K_1x06_P2.00mm_Vertical -> Connector_JST:JST_XH_B6B-XH-A_1x06_P2.50mm_Vertical; MPN B6B-PH-K-S(LF)(SN) -> B6B-XH-A

Commit message: Silk: J9 polarity text clear of BATT label; schematic fuse MPN synced (parity 0)
Co-Authored-By: Claude Opus 4.8 (1M context) <noreply@anthropic.com>
Parts:
- F1: MPN MINISMDC260F/16-2 -> MINISMDC350F/16-2
Changed lines of the file:
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@@
 			(effects (font (size 1.27 1.27)) (hide yes))
 		)
-		(property "MPN" "MINISMDC260F/16-2"
+		(property "MPN" "MINISMDC350F/16-2"
 			(at 90.17 149.86 0)
 			(effects (font (size 1.27 1.27)) (hide yes))

Commit message: Rev 7.2: XT60 + buzzer + ZH direct-plug motors + IMU self-test -- verify_drc 0/0, 12/12 battery, dual fab packages
User work order (HANDOFF 18) + same-day requests, all closed:
- J10 AMASS XT60-M (male) battery input in PARALLEL with J1 JST-XH:
  rear-right shelf placement via hole-aware free-rect scan against the
  true Edge.Cuts polygon with optical-corridor keepouts (two earlier
  candidate spots rejected with evidence: outline void / line-array
  through-holes). 0.8mm BATT_RAW feed; '+'/'-' + ONE PACK ONLY silk;
  normal BOM line (Lion procures; hand-fit fallback documented).
- BZ1 buzzer (CMT-8504, 15R coil) on IO46 via R81 220R -> Q34 MMBT2222A
  + D29 1N4148W flyback; strap-safe (load only ever pulls the boot strap
  low). fw beep API: ready/run/stop/low-batt/stall/IMU-fail chirps.
- J5/J6 -> JST ZH B6B-ZR in the robu GA12-N20 factory-cable order
  (M1,VCC,C1,C2,GND,M2): motor plugs straight in, zero soldering.
  Meter-check VCC/GND (pins 2/5) once before first plug-in.
- J9 balance lead now OPTIONAL: fw auto-detects (BAT_MID_SENSE ~0V) and
  falls back to the 6.6V pack floor.
- IMU functioning checks: sim_preflight I1-I6 (bus topology, Fast-mode
  timing, straps, reset pull-ups, CAP, INT, register audit) + boot
  self-test in fw (CHIP_ID, POST, fusion status; 4-chirp on failure).
- Sims updated to the exact ordered motor (600 ticks/rev, 200RPM, 43mm
  wheel, 0.23A stall); 8.4V question closed: motors sit on the regulated
  6.00V rail (circuit_tests M2/M3).
- Selective silk refdes for 23 debug-critical parts (clear-spot scanner
  seeded against board labels) + assembly-top/bottom.pdf debug maps
  (new export_fab gate). Project-local 3D models for ZH + buzzer.
- Production folders (pcb/tools/export_release.py): fab_release/
  lion-circuits/ (gerber zip + BOM + pos + assembly PDFs + ORDERING.md)
  and fab_release/jlcpcb/ (flat gerber+drill zip, JLC-format BOM/CPL,
  ORDERING.md with LCSC/rotation/origin caveats).
- Full Lion stock re-sweep 2026-07-19/20: every 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
Parts:
- added BZ1: CMT-8504-100-SMT (magnetic transducer 8.5mm, 15R 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, Buzzer_Beeper:MagneticBuzzer_CUI_CMT-8504-100-SMT, symbol Device:Buzzer
- added D29: 1N4148W (flyback clamp across the buzzer coil), Diode_SMD:D_SOD-123, symbol Device:D
- added J10: BATT_IN_XT60 (parallel option -- ONE PACK ONLY), Connector_AMASS:AMASS_XT60-M_1x02_P7.20mm_Vertical, symbol Connector_Generic:Conn_01x02
- added Q34: MMBT2222A (buzzer low-side driver; Q_NPN_BEC base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, Package_TO_SOT_SMD:SOT-23, symbol Transistor_BJT:Q_NPN_BEC
- added R81: 220, Resistor_SMD:R_0805_2012Metric, symbol Device:R
- J5, J6: footprint Connector_JST:JST_XH_B6B-XH-A_1x06_P2.50mm_Vertical -> Connector_JST:JST_ZH_B6B-ZR_1x06_P1.50mm_Vertical; MPN B6B-XH-A -> B6B-ZR(LF)(SN)
Connections:
- net BATT_RAW: now also J10.1 (Pin_1)
- net ENC1_A: now also J5.3 (Pin_3); no longer J5.5 (Pin_5)
- net ENC1_B: now also J5.4 (Pin_4); no longer J5.6 (Pin_6)
- net ENC2_A: now also J6.3 (Pin_3); no longer J6.5 (Pin_5)
- net ENC2_B: now also J6.4 (Pin_4); no longer J6.6 (Pin_6)
- net GND: now also J5.2 (Pin_2), J5.5 (Pin_5), J6.2 (Pin_2), J6.5 (Pin_5), BZ1.1 (+), D29.1 (K), J10.2 (Pin_2), Q34.2 (E); no longer J5.3 (Pin_3), J5.4 (Pin_4), J6.3 (Pin_3), J6.4 (Pin_4)
- net MOTA_N: now also J5.6 (Pin_6); no longer J5.2 (Pin_2)
- net MOTB_N: now also J6.6 (Pin_6); no longer J6.2 (Pin_2)
- net BUZZ_CTRL: now reaches U3.16 (IO46)
- net BUZZ_CTRL: now also R81.1
- new net: Q34.1 (B), R81.2
- new net BUZZ_DRV: BZ1.2 (-), D29.2 (A), Q34.3 (C)
- no-connect marks 13 -> 12
Other:
- note added: "10k pull-ups on all 4 encoder lines -- defensive: N20-encoder wire-color-to- function mapping is unverified for the exact unit ordered (see PROJECT_NOTES.md), and encoder output stage (open-drain vs push-pull) isn't confirmed either. A pull-up is required if open-drain and harmless if push-pull. Rev 7.2: J5/J6 are JST ZH B6B-ZR in the ROBU CABLE order (M1,VCC,C1,C2,GND,M2) -- the motor's factory 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"
- note added: "ESP32-S3-WROOM-1 on FreeRTOS: 6 wall sensors DIRECT on ADC1 IO1-IO6 (a fired pair is sampled in parallel), line array via U4 (IO7 + IO11-13), battery IO8, TB6612 on IO9/10/38/45, buzzer IO46 (straps 45/46 = idle-low outputs ONLY -- never add pull-ups), encoders IO43/44/47/48 (PCNT hardware quadrature via GPIO matrix), JTAG on the real JTAG quad IO39-42 -> J8 (ESP-Prog). Buttons: SW1=IO0 (start/BO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"
- note removed: "10k pull-ups on all 4 encoder lines -- defensive: N20-encoder wire-color-to- function mapping is unverified for the exact unit ordered (see PROJECT_NOTES.md), and encoder output stage (open-drain vs push-pull) isn't confirmed either. A pull-up is required if open-drain and harmless if push-pull. Motor connector pin order is FUNCTIONAL (M+,M-,ENC_VCC,ENC_GND,ENC_A,ENC_B) -- verify against the real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"
- note removed: "ESP32-S3-WROOM-1 on FreeRTOS: 6 wall sensors DIRECT on ADC1 IO1-IO6 (a fired pair is sampled in parallel), line array via U4 (IO7 + IO11-13), battery IO8, TB6612 on IO9/10/18/21/38/45/46 (straps 45/46 = idle-low outputs ONLY -- never add pull-ups), encoders IO43/44/47/48 (PCNT hardware quadrature via GPIO matrix), JTAG on the real JTAG quad IO39-42 -> J8 (ESP-Prog). Buttons: SW1=IO0 (start/BOOT),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"
