File: tht-assembly/pcb/micromouse-tht.kicad_sch (KiCad schematic)
At the start: 156 parts, among them J1 BATT_IN_2S (XH), J10 BATT_IN_XT60 (parallel -- ONE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, J11 TB6612_SIGNALS (PWMA,AIN2,AIN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, J12 TB6612_POWER (VM,VCC,GND,A01,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, J13 DEVKIT_LEFT, J14 DEVKIT_RIGHT, J15 GY-BNO055 (VIN,GND,SCL,SDA,IN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, J5 MOTOR_A (M1,VCC,C1,C2,GND,M2), J6 MOTOR_B (M1,VCC,C1,C2,GND,M2), J8 JTAG_1x6, J9 BALANCE_2S (optional), Q1 IRF9540N (TO-220 G-D-S revers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, Q121 BS250P (TO-92 D-G-S), Q122 BS250P (TO-92 D-G-S), Q123 BS250P (TO-92 D-G-S), Q124 BS250P (TO-92 D-G-S), Q125 BS250P (TO-92 D-G-S), Q126 BS250P (TO-92 D-G-S), Q131 BS250P (TO-92 D-G-S), Q132 BS250P (TO-92 D-G-S), Q133 BS250P (TO-92 D-G-S), Q134 BS250P (TO-92 D-G-S), Q135 BS250P (TO-92 D-G-S), Q136 BS250P (TO-92 D-G-S), Q137 BS250P (TO-92 D-G-S), Q138 BS250P (TO-92 D-G-S), Q16 2N7000 (TO-92 S-G-D), Q17 2N7000 (TO-92 S-G-D), Q18 2N7000 (TO-92 S-G-D), Q19 2N7000 (TO-92 S-G-D), Q2 PT334-6B (SFH309 base symbol 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, Q3 PT334-6B (SFH309 base symbol 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, Q34 PN2222A (TO-92 E-B-C), Q35 2N7000 (TO-92 S-G-D), Q4 PT334-6B (SFH309 base symbol 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, Q5 PT334-6B (SFH309 base symbol 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, Q6 PT334-6B (SFH309 base symbol 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, Q7 PT334-6B (SFH309 base symbol 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, SW1 BTN_A (start/BOOT), SW2 RESET, SW3 BTN_B, SW4 BTN_C, SW5 PWR ALL (EG1218; toward GND =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, SW6 PWR MOTORS (EG1218; toward GN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, U1 LM2596T-3.3 (TO-220-5), U4 CD74HC4067E (DIP-24 in socket), U7 LM2596T-ADJ -> 6.0V (TO-220-5)

Commit message: THT assembly M3: full placement converged -- 156 parts, 0 overlaps, 448 pins mapped
build_pcb_tht.py v11: SMD-verified optic geometry copied verbatim; DevKitC-1
socket rows across the rear (antenna notch removed from the outline -- the
DevKit antenna rides above); CD74HC4067E DIP flat under the DevKit deck;
TB6612 breakout rows horizontal at the right edge clear of the side-optic
corridor; all 66 axial resistors + 20 TO-92s + piezo + flyback on the BOTTOM
face grids (inside the ride-height budget), leaving the top face for optics,
power ranks (greedy-packed by measured courtyards), LEDs, buttons and
connectors. GND F/B/In1 + 3V3 In2 planes. Iteration trail v4->v11 in git.

Co-Authored-By: Claude Fable 5 <noreply@anthropic.com>
Parts:
- D30, D31: footprint Diode_THT:D_DO-201AD_P12.70mm_Horizontal -> Diode_THT:D_DO-201AD_P5.08mm_Vertical_CathodeUp
- U4: value CD74HC4067E (DIP-24 in socket) -> CD74HC4067E (DIP-24, soldered flat -- sits under the DevKit); footprint Package_DIP:DIP-24_W15.24mm_Socket -> Package_DIP:DIP-24_W15.24mm

Commit message: THT placement CLEAN: 0 courtyard overlaps (line array removed, 2 RGB LEDs added, JTAG dropped)
Per user: removed the line-follower array + mux (~50 parts -> board decongested
198->145 parts), added 2x ESP-driven common-cathode RGB LEDs (D40/D41,
Kingbright WP154A4, 6 LEDC channels via freed pins), dropped the redundant
external JTAG header (DevKit has USB-JTAG). DevKit socket recentred (x25.5) to
sit between the motor-bracket holes. Optic courtyards shrunk to body-true
circles (r=2.4) so the 45-deg diagonal emitter/detector pairs clear DRC.
verify_drc courtyard overlaps: 0. Next: route + DRC gate.

Co-Authored-By: Claude Fable 5 <noreply@anthropic.com>
Parts:
- removed D131, D132, D133, D134, D135, D136, D137, D138: LED red 3mm, LED_THT:LED_D3.0mm, symbol Device:D
- removed J8: JTAG_1x6, Connector_PinHeader_2.54mm:PinHeader_1x06_P2.54mm_Vertical, symbol Connector_Generic:Conn_01x06
- removed LS1, LS2, LS3, LS4, LS5, LS6, LS7, LS8: TCRT5000 (PC817 base symbol so ERC checks pins), n20:TCRT5000, symbol Isolator:PC817
- removed Q131, Q132, Q133, Q134, Q135, Q136, Q137, Q138: BS250P (TO-92 D-G-S), Package_TO_SOT_THT:TO-92_Inline, symbol Transistor_FET:Q_PMOS_DGS
- removed Q19: 2N7000 (TO-92 S-G-D), Package_TO_SOT_THT:TO-92_Inline, symbol Transistor_FET:Q_NMOS_SGD
- removed R101, R102, R103, R104, R105, R106, R107, R108: 120, Resistor_THT:R_Axial_DIN0207_L6.3mm_D2.5mm_P10.16mm_Horizontal, symbol Device:R
- removed R111, R112, R113, R114, R115, R116, R117, R118: 47k, Resistor_THT:R_Axial_DIN0207_L6.3mm_D2.5mm_P10.16mm_Horizontal, symbol Device:R
- removed R161, R162, R163, R164, R165, R166, R167, R168: 1k, Resistor_THT:R_Axial_DIN0207_L6.3mm_D2.5mm_P10.16mm_Horizontal, symbol Device:R
- removed R61: 100k, Resistor_THT:R_Axial_DIN0207_L6.3mm_D2.5mm_P10.16mm_Horizontal, symbol Device:R
- removed U4: CD74HC4067E (DIP-24, soldered flat -- sits under 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, Package_DIP:DIP-24_W15.24mm, symbol 74xx:CD74HC4067M
- added D40, D41: WP154A4SUREQBFZGC (5mm common-cathode RGB), LED_THT:LED_D5.0mm-4_RGB, symbol Device:LED_RKGB
- added R201, R204: 180, Resistor_THT:R_Axial_DIN0207_L6.3mm_D2.5mm_P10.16mm_Horizontal, symbol Device:R
- added R202, R203, R205, R206: 68, Resistor_THT:R_Axial_DIN0207_L6.3mm_D2.5mm_P10.16mm_Horizontal, symbol Device:R
Connections:
- net MUX_S3 is gone; now on net BAT_MID_SENSE: J13.12 (Pin_12)
- net MUX_SENSE is gone; now on net VBAT_SENSE: J13.7 (Pin_7)
- net GND: now also D40.2 (K), D41.2 (K)
- net RGB2_G: now reaches J13.21 (Pin_21)
- net RGB2_G: now also R205.1
- net JTAG_TCK: no longer names the net of J14.9 (Pin_9)
- net JTAG_TDI: no longer names the net of J14.7 (Pin_7)
- net JTAG_TDO: no longer names the net of J14.8 (Pin_8)
- net JTAG_TMS renamed RGB2_B
- net RGB2_B: now also R206.1
- net LINE_EMIT renamed RGB2_R
- net RGB2_R: now also R204.1
- net MUX_S0 renamed RGB1_R
- net RGB1_R: now also R201.1
- net MUX_S1 renamed RGB1_G
- net RGB1_G: now also R202.1
- net MUX_S2 renamed RGB1_B
- net RGB1_B: now also R203.1
- new net RGB1_BA: D40.4 (BA), R203.2
- new net RGB1_GA: D40.3 (GA), R202.2
- new net RGB1_RA: D40.1 (RA), R201.2
- new net RGB2_BA: D41.4 (BA), R206.2
- new net RGB2_GA: D41.3 (GA), R205.2
- new net RGB2_RA: D41.1 (RA), R204.2
- no-connect marks 10 -> 6
Other:
- note added: "INDICATORS -- LED ON = wall seen: 6 wall channels (BS250P + 1k + 3mm LED)"
- note removed: "INDICATORS -- LED ON = seen: 6 wall + 8 line channels (BS250P + 1k + 3mm LED)"
- note removed: "LINE ARRAY -- 8x TCRT5000 through CD74HC4067E (DIP-24 socket) + battery telemetry"
