File: pcb/JLCPCB_2layers_simplified/xiao_linefollower/design/micromouse-pcb-simplified-2l.kicad_pcb (KiCad board)
At the start: 2 copper layers, 100 x 120 mm, 73 parts, among them J1 JST_XH_B2B-XH-A_1x02_P2.50mm_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, J10 AMASS_XT60-M_1x02_P7.20mm_Ver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, J5 JST_ZH_B6B-ZR_1x06_P1.50mm_Ve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, J6 JST_ZH_B6B-ZR_1x06_P1.50mm_Ve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, Q1 SOT-23, Q16 SOT-23, Q17 SOT-23, Q18 SOT-23, Q2 LED_D5.0mm_IRBlack, Q3 LED_D5.0mm_IRBlack, Q34 SOT-23, Q4 LED_D5.0mm_IRBlack, Q5 LED_D5.0mm_IRBlack, Q6 LED_D5.0mm_IRBlack, Q7 LED_D5.0mm_IRBlack, SW1 SW_Push_1P1T_NO_CK_KMR2, SW2 SW_Push, SW5 SW_SPDT_PCM12, SW6 MOTOR KILL (PCM12), U1 TSOT-23-6, U2 SSOP-24_5.3x8.2mm_P0.65mm, U3 XIAO-nRF52840-Plus-SMD

Commit message: xiao 2L: power net closed, stale production package removed, comments corrected
- Net-(Q1-D) (fuse -> reverse-polarity FET, full battery current) is now routed
  at 0.5mm. Zero signal nets remain open.
- DELETED production_2layer/{jlcpcb,lioncircuits} contents. They were generated
  2026-08-05, BEFORE the XIAO pad-map defect was found, so they encoded the
  fatal wiring (pin 12 3V3_OUT shorted to GND, pin 13 GND floating). A stale
  gerber zip in a folder named "production" is an accident waiting to happen;
  DO_NOT_ORDER.md replaces them and explains how to regenerate.
- Deleted the two renders for the same reason (they show the pre-fix board).
- Corrected the last 5 stale pad-map comments in build_schematic.py, which still
  claimed pad12=GND/pad13=5V/pad14=3V3 and described the map as an ASSUMPTION.
  They now carry the verified map, the md5 evidence, and the D14/D15/D16
  restrictions. That contradiction is exactly how the bug would come back.

Verification of this state:
  vendor DRC (JLC-cap-Lion, all severities) .... 0
  schematic parity ............................. 0
  ERC (all severities) ......................... 0
  IPC audit .................................... PASS + 2 advisories
  unconnected .................................. 4 (all GND pour islands)

STILL OPEN -- 3 ground pads reach only isolated pour islands:
  U2 pad 18 (TB6612 logic ground)  legal via at (48.99,33.13) 2.35mm away
  C8 pad 2  (XIAO 3V3 decoupling)  legal via at (68.05,107.48) 3.10mm away
  R63 pad 2 (emitter gate pulldown) legal via at (55.91,48.02) 2.20mm away
Legal via positions exist and are listed above (verified against the full
vendor rule set); what fails is the headless A* escaping the pad through
congested copper. KiCad's interactive push-and-shove router closes these in
minutes -- that is the right tool, not more autorouter cycles.

Do NOT fabricate until those 3 are connected: a floating logic ground on the
motor driver and missing decoupling return are functional faul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
Routing:
- net Net-(Q1-D): track 0.00 -> 106.1 mm, vias 0 -> 6
Changed lines of the file:
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@@
+	)
+	(segment
+		(start 16.6 53.199999)
+		(end 16.6 51.6)
+		(width 0.5)
+		(layer "F.Cu")
+		(net "Net-(Q1-D)")
+	)
+	(segment
+		(start 16.6 51.6)
+		(end 15.8 50.8)
+		(width 0.5)
+		(layer "F.Cu")
+		(net "Net-(Q1-D)")
+	)
+	(segment
+		(start 30.4 35.4)
+		(end 30.4 36.8)
+		(width 0.5)
+		(layer "F.Cu")
+		(net "Net-(Q1-D)")
+	)
+	(segment
+		(start 23 31.4)
+		(end 24.599999 33)
+		(width 0.5)
+		(layer "F.Cu")
+		(net "Net-(Q1-D)")
+	)
+	(segment
+		(start 35.4 100.638)
+		(end 35.4 97.4)
+		(width 0.5)
+		(layer "F.Cu")
+		(net "Net-(Q1-D)")
+	)
+	(segment
+		(start 36.8 37.6)
+		(end 36.7 37.5)
+		(width 0.5)
+		(layer "F.Cu")
+		(net "Net-(Q1-D)")
+	)
+	(segment
+		(start 37.4 93.4)
+		(end 38.4 92.4)
+		(width 0.5)
+		(layer "F.Cu")
+		(net "Net-(Q1-D)")
+	)
+	(segment
+		(start 24.599999 33)
+		(end 28 33)
+		(width 0.5)
+		(layer "F.Cu")
+		(net "Net-(Q1-D)")
+	)
+	(segment
+		(start 34.938 101.1)
+		(end 35.4 100.638)
+		(width 0.5)
+		(layer "F.Cu")
+		(net "Net-(Q1-D)")
+	)
+	(segment
+		(start 38.4 75)
+		(end 16.6 53.199999)
+		(width 0.5)
+		(layer "F.Cu")
+		(net "Net-(Q1-D)")
+	)
+	(segment
+		(start 36.7 37.5)
+		(end 36.638 37.5)
+		(width 0.5)
+		(layer "F.Cu")
+		(net "Net-(Q1-D)")
+	)
+	(segment
+		(start 28 33)
+		(end 30.4 35.4)
+		(width 0.5)
+		(layer "F.Cu")
+		(net "Net-(Q1-D)")
+	)
+	(segment
+		(start 38.4 92.4)
+		(end 38.4 75)
+		(width 0.5)
+		(layer "F.Cu")
+		(net "Net-(Q1-D)")
+	)
+	(via
+		(at 30.4 36.8)
+		(size 0.6)
+		(drill 0.3)
+		(layers "F.Cu" "B.Cu")
+		(net "Net-(Q1-D)")
+	)
+	(via
+		(at 37.4 93.4)
+		(size 0.6)
+		(drill 0.3)
+		(layers "F.Cu" "B.Cu")
+		(net "Net-(Q1-D)")
+	)
+	(via
+		(at 23 31.4)
+		(size 0.6)
+		(drill 0.3)
+		(layers "F.Cu" "B.Cu")
+		(net "Net-(Q1-D)")
+	)
+	(via
+		(at 15.8 50.8)
+		(size 0.6)
+		(drill 0.3)
+		(layers "F.Cu" "B.Cu")
+		(net "Net-(Q1-D)")
+	)
+	(via
+		(at 36.8 37.6)
+		(size 0.6)
+		(drill 0.3)
+		(layers "F.Cu" "B.Cu")
+		(net "Net-(Q1-D)")
+	)
+	(via
+		(at 35.4 97.4)
+		(size 0.6)
+		(drill 0.3)
+		(layers "F.Cu" "B.Cu")
+		(net "Net-(Q1-D)")
+	)
+	(segment
+		(start 35.4 97.4)
+		(end 37.4 95.4)
+		(width 0.5)
+		(layer "B.Cu")
+		(net "Net-(Q1-D)")
+	)
+	(segment
+		(start 15.8 50.8)
+		(end 11.6 46.6)
+		(width 0.5)
+		(layer "B.Cu")
+		(net "Net-(Q1-D)")
+	)
+	(segment
+		(start 11.8 41.4)
+		(end 13.6 39.6)
+		(width 0.5)
+		(layer "B.Cu")
+		(net "Net-(Q1-D)")
+	)
+	(segment
+		(start 20.8 33.6)
+		(end 23 31.4)
+		(width 0.5)
+		(layer "B.Cu")
+		(net "Net-(Q1-D)")
+	)
+	(segment
+		(start 30.4 36.8)
+		(end 31.2 37.6)
+		(width 0.5)
+		(layer "B.Cu")
+		(net "Net-(Q1-D)")
+	)
+	(segment
+		(start 37.4 95.4)
+		(end 37.4 93.4)
+		(width 0.5)
+		(layer "B.Cu")
+		(net "Net-(Q1-D)")
+	)
+	(segment
+		(start 13.6 39.6)
+		(end 16.6 39.6)
+		(width 0.5)
+		(layer "B.Cu")
+		(net "Net-(Q1-D)")
+	)
+	(segment
+		(start 11.8 43.4)
+		(end 11.8 41.4)
+		(width 0.5)
+		(layer "B.Cu")
+		(net "Net-(Q1-D)")
+	)
+	(segment
+		(start 16.6 39.6)
+		(end 20.8 35.4)
+		(width 0.5)
+		(layer "B.Cu")
+		(net "Net-(Q1-D)")
+	)
+	(segment
+		(start 11.6 43.6)
+		(end 11.8 43.4)
+		(width 0.5)
+		(layer "B.Cu")
+		(net "Net-(Q1-D)")
+	)
+	(segment
+		(start 20.8 35.4)
+		(end 20.8 33.6)
+		(width 0.5)
+		(layer "B.Cu")
+		(net "Net-(Q1-D)")
+	)
+	(segment
+		(start 11.6 46.6)
+		(end 11.6 43.6)
+		(width 0.5)
+		(layer "B.Cu")
+		(net "Net-(Q1-D)")
+	)
+	(segment
+		(start 31.2 37.6)
+		(end 36.8 37.6)
+		(width 0.5)
+		(layer "B.Cu")
+		(net "Net-(Q1-D)")
 	)
 	(segment
